File: hardware/pcb/four-tone-driver.kicad_sch (KiCad schematic)
At the start: 55 parts, among them J1 PWR 12V/5V, J11 B2B-XH-A, J12 B2B-XH-A, J13 B2B-XH-A, J14 B2B-XH-A, J15 B2B-XH-A, J16 B2B-XH-A, J2 Socket 1x15, J3 Socket 1x15, Q1 AO3400A, Q2 AO3400A, Q3 AO3400A, Q4 AO3400A, Q5 AO3400A, Q6 AO3400A

Commit message: Lay out the six fan driver, rev A
- Routed 2-layer board, 130 x 70 mm: fan headers along the bottom edge,
  power terminal on the left edge, Nano sockets top right with the USB
  end at the right edge; GND pours on both layers with stitching vias
- Channels remapped to follow the Nano header order so gate traces do
  not cross: CH1 D3/J11, CH2 D5/J12, CH3 D6/J13, CH4 D9/J14,
  CH5 D10/J15, CH6 D11/J16
- Firmware pipes 1-4 now drive channels 1-4 (pins 3, 5, 6, 9)
- Board renamed six fan driver; silkscreen carries the licence and the
  CERN-OHL-S source location github.com/ideocentric/four-tone, also in
  the schematic title block and LICENSE.md
- Silkscreen: FAN labels on the edge side of the headers, outline of the
  Nano's USB connector for orientation, and the enso house mark
- Enso artwork committed as source in hardware/art/ (copied from
  caryatid, first party)
- ERC and DRC clean, 0 unconnected, 0 schematic parity issues
Connections:
- net FAN1_PWM: now also A1.6 (D3), J2.6 (Pin_6); no longer A1.13 (D10), J2.13 (Pin_13)
- net FAN2_PWM: now also A1.8 (D5), J2.8 (Pin_8); no longer A1.12 (D9), J2.12 (Pin_12)
- net FAN4_PWM: now also A1.12 (D9), J2.12 (Pin_12); no longer A1.8 (D5), J2.8 (Pin_8)
- net FAN5_PWM: now also A1.13 (D10), J2.13 (Pin_13); no longer A1.6 (D3), J2.6 (Pin_6)
Other:
- note added: "CHANNEL 1 (Nano D3, connector J11)"
- note added: "CHANNEL 2 (Nano D5, connector J12)"
- note added: "CHANNEL 4 (Nano D9, connector J14)"
- note added: "CHANNEL 5 (Nano D10, connector J15)"
- note added: "six fan driver board"
- note removed: "CHANNEL 1 (Nano D10, connector J11)"
- note removed: "CHANNEL 2 (Nano D9, connector J12)"
- note removed: "CHANNEL 4 (Nano D5, connector J14)"
- note removed: "CHANNEL 5 (Nano D3, connector J15)"
- note removed: "four-tone fan driver board"
- company: four-tone -> four-tone project
- title: four-tone fan driver -> six fan driver
Changed lines of the file:
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@@
 	(paper "A3")
 	(title_block
-		(title "four-tone fan driver")
+		(title "six fan driver")
 		(date "2026-09-15")
 		(rev "A")
-		(company "four-tone")
+		(company "four-tone project")
 		(comment 1 "CERN-OHL-S-2.0")
 		(comment 2 "Parts: JLCPCB/LCSC numbers in the LCSC field")
+		(comment 3 "Source: https://github.com/ideocentric/four-tone")
 	)
-	(text "four-tone fan driver board"
+	(text "six fan driver board"
 		(exclude_from_sim no)
 		(at 25.4 22.86 0)
@@
 		(stroke (width 0) (type default))
 	)
-	(label "FAN5_PWM"
+	(label "FAN1_PWM"
 		(at 149.86 81.28 180)
 		(effects (font (size 1.27 1.27)) (justify right bottom))
@@
 		(stroke (width 0) (type default))
 	)
-	(label "FAN4_PWM"
+	(label "FAN2_PWM"
 		(at 149.86 86.36 180)
 		(effects (font (size 1.27 1.27)) (justify right bottom))
@@
 		(stroke (width 0) (type default))
 	)
-	(label "FAN2_PWM"
+	(label "FAN4_PWM"
 		(at 149.86 96.52 180)
 		(effects (font (size 1.27 1.27)) (justify right bottom))
@@
 		(stroke (width 0) (type default))
 	)
-	(label "FAN1_PWM"
+	(label "FAN5_PWM"
 		(at 149.86 99.06 180)
 		(effects (font (size 1.27 1.27)) (justify right bottom))
@@
 		(stroke (width 0) (type default))
 	)
-	(label "FAN5_PWM"
+	(label "FAN1_PWM"
 		(at 213.36 83.82 180)
 		(effects (font (size 1.27 1.27)) (justify right bottom))
@@
 		(stroke (width 0) (type default))
 	)
-	(label "FAN4_PWM"
+	(label "FAN2_PWM"
 		(at 213.36 88.9 180)
 		(effects (font (size 1.27 1.27)) (justify right bottom))
@@
 		(stroke (width 0) (type default))
 	)
-	(label "FAN2_PWM"
+	(label "FAN4_PWM"
 		(at 213.36 99.06 180)
 		(effects (font (size 1.27 1.27)) (justify right bottom))
@@
 		(stroke (width 0) (type default))
 	)
-	(label "FAN1_PWM"
+	(label "FAN5_PWM"
 		(at 213.36 101.6 180)
 		(effects (font (size 1.27 1.27)) (justify right bottom))
@@
 		(effects (font (size 1.27 1.27) (bold yes)) (justify left bottom))
 	)
-	(text "CHANNEL 1  (Nano D10, connector J11)"
+	(text "CHANNEL 1  (Nano D3, connector J11)"
 		(exclude_from_sim no)
 		(at 25.4 144.78 0)
@@
 		(effects (font (size 1.27 1.27)) (justify right bottom))
 	)
-	(text "CHANNEL 2  (Nano D9, connector J12)"
+	(text "CHANNEL 2  (Nano D5, connector J12)"
 		(exclude_from_sim no)
 		(at 149.86 144.78 0)
@@
 		(effects (font (size 1.27 1.27)) (justify right bottom))
 	)
-	(text "CHANNEL 4  (Nano D5, connector J14)"
+	(text "CHANNEL 4  (Nano D9, connector J14)"
 		(exclude_from_sim no)
 		(at 25.4 205.74 0)
@@
 		(effects (font (size 1.27 1.27)) (justify right bottom))
 	)
-	(text "CHANNEL 5  (Nano D3, connector J15)"
+	(text "CHANNEL 5  (Nano D10, connector J15)"
 		(exclude_from_sim no)
 		(at 149.86 205.74 0)
